File: oddball.kicad_pcb (KiCad board)
At the start: 2 copper layers, 176.7 x 84.4 mm, 62 parts, among them J1 Conn_01x03, J2 Conn_01x03, J3 TRRS, J4 Conn_02x04_Counter_Clockwise, J5 Conn_02x04_Counter_Clockwise, SW1 KEYSW, SW10 KEYSW, SW11 KEYSW, SW12 KEYSW, SW13 KEYSW, SW14 KEYSW, SW15 KEYSW, SW16 KEYSW, SW17 KEYSW, SW18 KEYSW, SW19 KEYSW, SW2 KEYSW, SW20 KEYSW, SW21 KEYSW, SW3 KEYSW, SW4 KEYSW, SW5 KEYSW, SW6 KEYSW, SW7 KEYSW, SW8 KEYSW, SW9 KEYSW, U1 ELITEC, U4 HOLE

Commit message: simple panel
Parts:
- added REF**: PerfHole, oddball:PerfHole, F.Cu at (135.7, 111.8)
- added REF**: PerfHole, oddball:PerfHole, F.Cu at (97.4, 121.6)
- added REF**: PerfHole, oddball:PerfHole, F.Cu at (135.7, 109.5)
- added REF**: PerfHole, oddball:PerfHole, F.Cu at (142.0, 111.8)
- added REF**: PerfHole, oddball:PerfHole, F.Cu at (134.1, 111.8)
- added REF**: PerfHole, oddball:PerfHole, F.Cu at (140.4, 109.5)
- added REF**: PerfHole, oddball:PerfHole, F.Cu at (140.4, 111.8)
- added REF**: PerfHole, oddball:PerfHole, F.Cu at (142.0, 109.5)
- added REF**: PerfHole, oddball:PerfHole, F.Cu at (99.0, 116.5)
- added REF**: PerfHole, oddball:PerfHole, F.Cu at (134.1, 109.5)
- added REF**: PerfHole, oddball:PerfHole, F.Cu at (94.3, 116.5)
- added REF**: PerfHole, oddball:PerfHole, F.Cu at (137.2, 111.8)
- added REF**: PerfHole, oddball:PerfHole, F.Cu at (138.8, 111.8)
- added REF**: PerfHole, oddball:PerfHole, F.Cu at (102.1, 121.6)
- added REF**: PerfHole, oddball:PerfHole, F.Cu at (95.9, 116.5)
- added REF**: PerfHole, oddball:PerfHole, F.Cu at (95.8, 121.6)
- added REF**: PerfHole, oddball:PerfHole, F.Cu at (137.2, 109.5)
- added REF**: PerfHole, oddball:PerfHole, F.Cu at (94.2, 121.6)
- added REF**: PerfHole, oddball:PerfHole, F.Cu at (97.4, 116.5)
- added REF**: PerfHole, oddball:PerfHole, F.Cu at (100.5, 121.6)
- added REF**: PerfHole, oddball:PerfHole, F.Cu at (100.6, 116.5)
- added REF**: PerfHole, oddball:PerfHole, F.Cu at (99.0, 121.6)
- added REF**: PerfHole, oddball:PerfHole, F.Cu at (138.8, 109.5)
- added REF**: PerfHole, oddball:PerfHole, F.Cu at (102.2, 116.5)
- moved D21 142.8 mm to (99.8, 138.8), turned to 0 degrees
- moved SW21 141.1 mm to (99.8, 131.2), turned to 180 degrees
- moved D20 105.4 mm to (118.8, 138.8), turned to 0 degrees
- moved SW20 103.4 mm to (118.6, 131.1), turned to 180 degrees
- moved REF** 84.2 mm to (128.3, 122.7), turned to 180 degrees
- moved REF** 84.0 mm to (128.3, 130.6), turned to 180 degrees
- moved REF** 84.0 mm to (128.3, 124.3), turned to 180 degrees
- moved REF** 83.8 mm to (128.3, 129.0), turned to 180 degrees
- moved REF** 83.8 mm to (128.3, 125.8), turned to 180 degrees
- moved REF** 83.8 mm to (128.3, 127.4), turned to 180 degrees
- moved J2 76.2 mm to (134.6, 113.8), turned to -90 degrees
- moved SW19 66.0 mm to (137.7, 121.5), turned to 180 degrees
- moved D19 64.8 mm to (137.9, 129.3), turned to 0 degrees
Routing:
- net Net-(J2-Pin_1): track 3.84 -> 35.1 mm
- net row4: track 224.5 -> 237.5 mm
- net column6: track 89.4 -> 97.3 mm
- net Net-(D19-K): track 85.1 -> 80.4 mm
Other:
- board size 176.7 x 84.4 mm -> 109.3 x 83.3 mm
